Commit message: feat(grasp): spread bin objects and narrow gripper before descent
Move red_cylinder/yellow_box/brown_cube apart to ≥3.7cm edge-to-edge in
bin_scene.sdf so the gripper finger pads no longer clip a neighbor on
the way down, while keeping every center within ~0.40m of the base so
MoveIt can still plan to it.

Add a GRIPPER_APPROACH stage to the task state machine between
VERIFY_PREGRASP and MOVE_TO_GRASP. It commands the gripper to a partial
opening (default 0.010 → ~8.3cm gap, ~13.5cm outer pad span instead of
the ~15.5cm full-open span) so the finger pads stick out 1cm less per
side during the descent. The closing posture and place-time release are
unchanged.

Wire gripper_approach_position through task_demo.launch.py and refresh
README with the new bin layout, the approach stage, and the Nano +
RViz instructions.

Co-Authored-By: Claude Opus 4.7 <noreply@anthropic.com>

File: src/alicia_d_descriptions/urdf/Alicia_D_v5_6/Alicia_D_v5_6_gripper_100mm.urdf (robot description, URDF)
Before this commit: robot Alicia_D_v5_6_gripper_100mm, 10 links, 9 joints
Links:
- link left_gripper: geometry collision box size=0.070 0.070 0.026; visual mesh filename=package://alicia_d_descriptions/meshes/Alicia_D_v5_6/grippe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
- link right_gripper: geometry collision box size=0.070 0.070 0.026; visual mesh filename=package://alicia_d_descriptions/meshes/Alicia_D_v5_6/grippe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

File: src/alicia_moveit_config/config/alicia_d.ros2_control.xacro (robot description, xacro)
@@ -5,5 +5,5 @@
         Replaces the old fake_components/GenericSystem and real hardware xacro.
         Plugin: gz_ros2_control/GazeboSimSystem
-        Joints: Joint1~Joint6 (revolute) + Gripper (prismatic)
+        Joints: Joint1~Joint6 (revolute) + Gripper/right_finger (prismatic)
     -->
     <xacro:macro name="alicia_d_ros2_control" params="name initial_positions_file">
@@ -70,4 +70,13 @@
                 <state_interface name="velocity"/>
             </joint>
+            <!-- right_finger is a URDF mimic joint, but Gazebo physics still
+                 needs ros2_control to hold its real simulated joint. -->
+            <joint name="right_finger">
+                <command_interface name="effort"/>
+                <state_interface name="position">
+                    <param name="initial_value">${initial_positions['right_finger']}</param>
+                </state_interface>
+                <state_interface name="velocity"/>
+            </joint>
         </ros2_control>
         <gazebo>
