Commit message: fix(gripper): use effort PID control

File: src/alicia_d_descriptions/urdf/Alicia_D_v5_6/Alicia_D_v5_6_gripper_100mm.urdf (robot description, URDF)
Before this commit: robot Alicia_D_v5_6_gripper_100mm, 10 links, 9 joints
Links:
- link Link6: geometry visual mesh filename=package://alicia_d_descriptions/meshes/Alicia_D_v5_6/grippe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
- link left_gripper: geometry visual mesh filename=package://alicia_d_descriptions/meshes/Alicia_D_v5_6/grippe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
- link right_gripper: geometry visual mesh filename=package://alicia_d_descriptions/meshes/Alicia_D_v5_6/grippe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
Joints:
- joint Gripper: limit lower=0 upper=0.05 effort=5 velocity=12 -> lower=0 upper=0.05 effort=100 velocity=12
- joint right_finger: limit lower=-0.05 upper=0 effort=5 velocity=12 -> lower=-0.05 upper=0 effort=100 velocity=12

File: src/alicia_moveit_config/config/alicia_d.ros2_control.xacro (robot description, xacro)
@@ -64,5 +64,5 @@
             <!-- Gripper — Prismatic (parallel jaw, 0=open, 0.05=closed) -->
             <joint name="Gripper">
-                <command_interface name="position"/>
+                <command_interface name="effort"/>
                 <state_interface name="position">
                     <param name="initial_value">${initial_positions['Gripper']}</param>

Commit message: gripper-center

File: src/alicia_d_descriptions/urdf/Alicia_D_v5_6/Alicia_D_v5_6_gripper_100mm.urdf (robot description, URDF)
Before this commit: robot Alicia_D_v5_6_gripper_100mm, 10 links, 9 joints
Joints:
- joint finger: origin xyz=-0.0002 0 0.13048 rpy=0 0 0 -> xyz=-0.0002 0 0.10 rpy=0 0 0
