Commit message: fix perception node

File: src/alicia_moveit_config/config/Alicia_D_v5_6_gripper_100mm.urdf.xacro (robot description, xacro)
@@ -13,5 +13,5 @@
         <parent link="world"/>
         <child link="base_link"/>
-        <origin xyz="0.20 0 0" rpy="0 0 0"/>
+        <origin xyz="0 0 0" rpy="0 0 0"/>
     </joint>
     <!-- Instantiate gz_ros2_control hardware interface -->
